File: Hardware/PCB_SATELITES/PCB_SAT_01/PCB_SAT_01.kicad_pcb (KiCad board)
At the start: 2 copper layers, 41 parts, among them IC1 OPT3001DNPRQ1, IC2 OPT3001DNPRQ1, IC3 OPT3001DNPRQ1, IC4 OPT3001DNPRQ1, J1 MTJ-88ARX1-FSM-LG

Commit message: Actualizacion PCB SATELITE 1
Parts:
- removed R10, R11, R12, R4, R5, R6, R7, R8, R9: 10k, Resistor_SMD:R_0805_2012Metric
- moved C3 117.2 mm to (85.0, 113.2), turned to 90 degrees
- moved IC3 111.8 mm to (91.4, 117.7)
- moved IC4 95.2 mm to (115.5, 117.7)
- moved C4 92.9 mm to (122.0, 113.2), turned to 90 degrees
- moved IC2 81.7 mm to (115.5, 94.2)
- moved C2 76.6 mm to (122.0, 88.1), turned to 90 degrees
- moved R3 71.9 mm to (97.1, 90.2), turned to 0 degrees
- moved C1 68.3 mm to (85.0, 88.7), turned to -90 degrees
- moved R2 66.8 mm to (97.1, 87.7), turned to 0 degrees
- moved TP4_2 64.9 mm to (131.0, 111.2)
- moved IC1 63.0 mm to (91.4, 94.2)
- moved TP3_3 62.0 mm to (77.0, 114.7)
- moved R1 61.7 mm to (97.1, 85.2), turned to 0 degrees
- moved TP3_5 55.3 mm to (77.0, 121.7)
- moved TP3_4 55.0 mm to (77.0, 118.2)
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Connections:
- net Net-(IC1-INT) renamed /INT
- net Net-(IC1-SDA) renamed /SDA
- IC1 pad 4: Net-(IC1-SCL) -> /SCL
- IC2 pad 4: Net-(IC1-SCL) -> /SCL
- IC3 pad 4: Net-(IC1-SCL) -> /SCL
- IC4 pad 2: Net-(IC1-SCL) -> /SCL
- IC4 pad 4: Net-(IC1-SCL) -> /SCL
- J1 pad 6: GND -> /SCL
- J1 pad 8: Net-(IC1-SCL) -> GND
- R3 pad 2: Net-(IC1-SCL) -> /SCL
- TP1_3 pad 1: Net-(IC1-SCL) -> /SCL
- TP2_3 pad 1: Net-(IC1-SCL) -> /SCL
- TP3_3 pad 1: Net-(IC1-SCL) -> /SCL
- TP4_3 pad 1: Net-(IC1-SCL) -> /SCL
Other:
- board text added: "OPT3001DNPRQ1"
- board text added: "PCB SATELITE"

Commit message: Actualizacion PCB SATELITE 1
Parts:
- removed C2, C3, C4: 100n, Capacitor_SMD:C_0805_2012Metric
- removed TP2_1, TP2_2, TP2_3, TP2_4, TP2_5, TP3_1, TP3_2, TP3_3, TP3_4, TP3_5, TP4_1, TP4_2, TP4_3, TP4_4, TP4_5: TestPoint, TestPoint:TestPoint_Pad_D1.0mm
- added H1: MountingHole_2.2mm_M2_ISO14580_Pad, MountingHole:MountingHole_2.2mm_M2_ISO14580_Pad, F.Cu at (78.0, 54.0)
- added H2: MountingHole_2.2mm_M2_ISO14580_Pad, MountingHole:MountingHole_2.2mm_M2_ISO14580_Pad, F.Cu at (130.0, 54.0)
- added H3: MountingHole_2.2mm_M2_ISO14580_Pad, MountingHole:MountingHole_2.2mm_M2_ISO14580_Pad, F.Cu at (130.0, 125.0)
- added H4: MountingHole_2.2mm_M2_ISO14580_Pad, MountingHole:MountingHole_2.2mm_M2_ISO14580_Pad, F.Cu at (78.0, 125.0)
- moved R2 34.6 mm to (89.5, 53.9)
- moved R3 34.6 mm to (89.5, 56.4)
- moved C1 32.2 mm to (83.5, 56.5), turned to 180 degrees
- moved TP_SCL 25.2 mm to (82.2, 69.5)
- moved TP_INT 22.5 mm to (82.2, 75.8)
- moved TP_GND 21.1 mm to (82.2, 66.8)
- moved TP_VDD 20.6 mm to (82.2, 63.8)
- moved TP_SDA 18.7 mm to (82.2, 72.8)
- moved R1 17.9 mm to (108.0, 70.9), turned to 90 degrees
- renumbered TP1_2 to TP_GND, TP1_5 to TP_INT, TP1_4 to TP_SCL, TP1_3 to TP_SDA, TP1_1 to TP_VDD
Connections:
- TP_INT pad 1: /SDA -> /INT
- TP_SCL pad 1: /INT -> /SCL
- TP_SDA pad 1: /SCL -> /SDA
Routing:
- net /INT: track 0.00 -> 177.9 mm, vias 0 -> 4
- net /SCL: track 0.00 -> 160.9 mm, vias 0 -> 2
- net /SDA: track 0.00 -> 158.3 mm
- net VDD: track 0.00 -> 14.7 mm, vias 0 -> 8
- net GND: track 0.00 -> 12.7 mm, vias 0 -> 10
- added copper zone on In2.Cu, net GND
- added copper zone on B.Cu, net VDD
Other:
- board outline added: 60 x 79 mm
- copper layers 2 -> 4

Commit message: actualizacion pcb satelite
Parts:
- removed H1, H2, H3, H4: MountingHole_2.2mm_M2_ISO14580_Pad, MountingHole:MountingHole_2.2mm_M2_ISO14580_Pad
- added C2: 100n, Capacitor_SMD:C_0805_2012Metric, F.Cu at (82.0, 97.0)
- added C3: 100n, Capacitor_SMD:C_0805_2012Metric, F.Cu at (82.0, 100.0)
- added C4: 100n, Capacitor_SMD:C_0805_2012Metric, F.Cu at (82.0, 103.0)
- moved C1 38.7 mm to (87.0, 95.0), turned to -90 degrees
- renumbered TP_GND to TP_GND1, TP_INT to TP_INT1, TP_SCL to TP_SCL1, TP_SDA to TP_SDA1, TP_VDD to TP_VDD1
Routing:
- net GND: track 12.7 -> 10.1 mm, vias 10 -> 9
- net VDD: track 14.7 -> 12.7 mm

Commit message: actualizacion pcb satelite 1
Parts:
- removed TP_GND1, TP_INT1, TP_SCL1, TP_SDA1, TP_VDD1: TestPoint, TestPoint:TestPoint_Pad_D1.0mm
- added TP_GND: TestPoint, TestPoint:TestPoint_Pad_D1.0mm, F.Cu at (142.5, 108.5)
- added TP_INT: TestPoint, TestPoint:TestPoint_Pad_D1.0mm, F.Cu at (142.5, 99.5)
- added TP_SCL: TestPoint, TestPoint:TestPoint_Pad_D1.0mm, F.Cu at (142.5, 95.0)
- added TP_SDA: TestPoint, TestPoint:TestPoint_Pad_D1.0mm, F.Cu at (142.5, 90.5)
- added TP_VDD: TestPoint, TestPoint:TestPoint_Pad_D1.0mm, F.Cu at (142.5, 104.0)
- moved C4 59.8 mm to (133.8, 133.0)
- moved C2 52.1 mm to (133.9, 102.6)
- moved R2 46.6 mm to (126.5, 82.2)
- moved R3 43.7 mm to (126.5, 79.6)
- moved C3 37.8 mm to (100.5, 133.0)
- moved R1 23.1 mm to (126.5, 84.8), turned to 0 degrees
- moved IC4 21.3 mm to (133.8, 128.5), turned to 90 degrees
- moved IC2 18.8 mm to (133.8, 98.1), turned to 90 degrees
- moved C1 15.5 mm to (100.5, 102.6), turned to 0 degrees
- moved J1 14.4 mm to (120.6, 66.0)
- moved IC3 14.2 mm to (100.5, 128.6), turned to 90 degrees
- moved IC1 9.94 mm to (100.5, 98.1), turned to 90 degrees
Routing:
- net /SCL: track 160.9 -> 221.8 mm, vias 2 -> 3
- net /INT: track 177.9 -> 232.2 mm, vias 4 -> 6
- net /SDA: track 158.3 -> 181.2 mm, vias 0 -> 6
- net VDD: track 12.7 -> 34.2 mm, vias 8 -> 6
- net GND: track 10.1 -> 24.0 mm, vias 9 -> 61
- added copper zone on In1.Cu, net (none)
- added copper zone on F.Cu, net GND
Other:
- board size 60 x 79 mm -> 66.5 x 84.5 mm
- board text removed: "OPT3001DNPRQ1"
- board text removed: "PCB SATELITE"
