File: Hardware/PCB/PCB/Solar_Tracker_PCB_Main/IMU.kicad_sch (KiCad schematic)
At the start: 1 part, among them IC3 BNO085

Commit message: actualizacion de pcb (IMU)
Parts:
- added C1, C2, C3, C4, C5: C, symbol Device:C
- added R1, R2, R3, R4, R5: R, symbol Device:R
- added Y1: Crystal, symbol Device:Crystal
Connections:
- net IMU_CLKSEL0: now reaches IC3.10 (CLKSEL0)
- net IMU_NRST: now reaches IC3.11 (NRST)
- net IMU_INT: now reaches IC3.14 (H_INTN)
- net IMU_INT: now also R5.2
- net SAO: now reaches IC3.17 (SA0/H_MOSI_)
- net SAO: now also R1.1, R2.2
- net IMU_SCL: now reaches IC3.19 (H_SCL/SCK/RX)
- net IMU_SCL: now also R4.2
- net GND: now reaches IC3.2 (GND_1)
- net GND: now also IC3.25 (GND_2), IC3.5 (PS1), IC3.6 (PS0/WAKE), C1.2, C2.2, C3.2, C4.2, C5.2, R1.2
- net IMU_SDA: now reaches IC3.20 (H_SDA/H_MISO/TX_)
- net IMU_SDA: now also R3.2
- net X_OUT: now reaches IC3.26 (XOUT32/CLKSEL1)
- net X_OUT: now also C5.1, Y1.2
- net X_IN: now reaches IC3.27 (XIN32)
- net X_IN: now also C4.1, Y1.1
- net VDD: now reaches IC3.28 (VDDIO)
- net VDD: now also IC3.3 (VDD), C1.1, C2.1, R2.1, R3.1, R4.1, R5.1
- net IMU_BOOTN: now reaches IC3.4 (BOOTN)
- net CAP: now reaches IC3.9 (CAP)
- net CAP: now also C3.1
Other:
- note added: "CRYSTAL CONNECTION"
- note added: "PULLUP RESISTOR"
- moved on the sheet: IC3

Commit message: actualizacion pcb main
Connections:
- no-connect marks 0 -> 12
Other:
- note added: "PULL-UP RESISTOR"
- note removed: "PULLUP RESISTOR"
- moved on the sheet: IC3, R1

Commit message: actualizacion pcb main
Connections:
- net SAO renamed SA0
Changed lines of the file:
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@@
+	(wire
+		(pts
+			(xy 59.69 165.1) (xy 59.69 162.56)
+		)
+		(stroke
+			(width 0)
+			(type default)
+		)
+	)
 	(wire
 		(pts
@@
 	(wire
 		(pts
+			(xy 97.79 137.16) (xy 87.63 137.16)
+		)
+		(stroke
+			(width 0)
+			(type default)
+		)
+	)
+	(wire
+		(pts
 			(xy 33.02 124.46) (xy 36.83 124.46)
 		)
@@
 	(wire
 		(pts
+			(xy 97.79 119.38) (xy 87.63 119.38)
+		)
+		(stroke
+			(width 0)
+			(type default)
+		)
+	)
+	(wire
+		(pts
 			(xy 39.37 31.75) (xy 45.72 31.75)
 		)
@@
 	(wire
 		(pts
+			(xy 85.09 44.45) (xy 85.09 55.88)
+		)
+		(stroke
+			(width 0)
+			(type default)
+		)
+	)
+	(wire
+		(pts
 			(xy 93.98 44.45) (xy 93.98 52.07)
 		)
@@
 	(wire
 		(pts
-			(xy 30.48 121.92) (xy 36.83 121.92)
+			(xy 31.75 121.92) (xy 36.83 121.92)
 		)
 		(stroke
@@
 	(wire
 		(pts
+			(xy 97.79 121.92) (xy 87.63 121.92)
+		)
+		(stroke
+			(width 0)
+			(type default)
+		)
+	)
+	(wire
+		(pts
 			(xy 157.48 33.02) (xy 157.48 36.83)
 		)
@@
 	(wire
 		(pts
-			(xy 85.09 44.45) (xy 85.09 55.88)
-		)
-		(stroke
-			(width 0)
-			(type default)
+			(xy 31.75 134.62) (xy 36.83 134.62)
+		)
+		(stroke
+			(width 0)
+			(type default)
+		)
+	)
+	(wire
+		(pts
+			(xy 64.77 162.56) (xy 64.77 165.1)
+		)
+		(stroke
+			(width 0)
+			(type default)
+		)
+	)
+	(label "SA0"
+		(at 59.69 165.1 270)
+		(effects
+			(font
+				(size 1.27 1.27)
+			)
+			(justify right bottom)
 		)
 	)
 	(label "CAP"
-		(at 30.48 121.92 0)
+		(at 31.75 121.92 180)
+		(effects
+			(font
+				(size 1.27 1.27)
+			)
+			(justify right bottom)
+		)
+	)
+	(label "X_OUT"
+		(at 97.79 121.92 0)
+		(effects
+			(font
+				(size 1.27 1.27)
+			)
+			(justify left bottom)
+		)
+	)
+	(label "X_IN"
+		(at 24.13 31.75 90)
+		(effects
+			(font
+				(size 1.27 1.27)
+			)
+			(justify left bottom)
+		)
+	)
+	(label "SA0"
+		(at 186.69 45.72 180)
+		(effects
+			(font
+				(size 1.27 1.27)
+			)
+			(justify right bottom)
+		)
+	)
+	(label "X_IN"
+		(at 97.79 119.38 0)
 		(effects
 			(font
@@
 		)
 	)
+	(label "X_OUT"
+		(at 45.72 31.75 90)
+		(effects
+			(font
+				(size 1.27 1.27)
+			)
+			(justify left bottom)
+		)
+	)
+	(global_label "IMU_SCL"
+		(shape input)
+		(at 64.77 165.1 270)
+		(fields_autoplaced yes)
+		(effects
+			(font
+				(size 1.27 1.27)
+			)
+			(justify right)
+		)
+		(property "Intersheetrefs" "${INTERSHEET_REFS}"
+			(at 64.77 175.9471 90)
+			(effects
+				(font
+					(size 1.27 1.27)
+				)
+				(justify right)
+				(hide yes)
+			)
+		)
+	)
 	(global_label "IMU_NRST"
 		(shape input)
@@
 	(global_label "IMU_SDA"
 		(shape input)
+		(at 97.79 137.16 0)
+		(fields_autoplaced yes)
+		(effects
+			(font
+				(size 1.27 1.27)
+			)
+			(justify left)
+		)
+		(property "Intersheetrefs" "${INTERSHEET_REFS}"
+			(at 108.6976 137.16 0)
+			(effects
+				(font
+					(size 1.27 1.27)
+				)
+				(justify left)
+				(hide yes)
+			)
+		)
+	)
+	(global_label "IMU_INT"
+		(shape input)
+		(at 31.75 134.62 180)
+		(fields_autoplaced yes)
+		(effects
+			(font
+				(size 1.27 1.27)
+			)
+			(justify right)
+		)
+		(property "Intersheetrefs" "${INTERSHEET_REFS}"
+			(at 21.5076 134.62 0)
+			(effects
+				(font
+					(size 1.27 1.27)
+				)
+				(justify right)
+				(hide yes)
+			)
+		)
+	)
+	(global_label "IMU_SDA"
+		(shape input)
 		(at 119.38 55.88 0)
 		(fields_autoplaced yes)
@@
 		)
 	)
-	(hierarchical_label "H_SCL"
-		(shape input)
-		(at 93.98 52.07 180)
-		(effects
-			(font
-				(size 1.27 1.27)
-			)
-			(justify right)
-		)
-	)
-	(hierarchical_label "SAO"
-		(shape input)
-		(at 186.69 45.72 0)
-		(effects
-			(font
-				(size 1.27 1.27)
-			)
-			(justify left)
-		)
-	)
-	(hierarchical_label "X_IN"
-		(shape input)
-		(at 87.63 119.38 0)
-		(effects
-			(font
-				(size 1.27 1.27)
-			)
-			(justify left)
-		)
-	)
-	(hierarchical_label "H_INTN"
-		(shape input)
-		(at 36.83 134.62 180)
-		(effects
-			(font
-				(size 1.27 1.27)
-			)
-			(justify right)
-		)
-	)
-	(hierarchical_label "H_SDA"
-		(shape input)
-		(at 87.63 137.16 0)
-		(effects
-			(font
-				(size 1.27 1.27)
-			)
-			(justify left)
-		)
-	)
-	(hierarchical_label "H_INTN"
-		(shape input)
-		(at 102.87 48.26 180)
-		(effects
-			(font
-				(size 1.27 1.27)
-			)
-			(justify right)
-		)
-	)
-	(hierarchical_label "X_IN"
-		(shape input)
-		(at 24.13 31.75 90)
-		(effects
-			(font
-				(size 1.27 1.27)
-			)
-			(justify left)
-		)
-	)
-	(hierarchical_label "H_SDA"
-		(shape input)
-		(at 85.09 55.88 180)
-		(effects
-			(font
-				(size 1.27 1.27)
-			)
-			(justify right)
-		)
-	)
-	(hierarchical_label "X_OUT"
-		(shape input)
-		(at 87.63 121.92 0)
-		(effects
-			(font
-				(size 1.27 1.27)
-			)
-			(justify left)
-		)
-	)
-	(hierarchical_label "H_SCL"
-		(shape input)
-		(at 64.77 162.56 270)
-		(effects
-			(font
-				(size 1.27 1.27)
-			)
-			(justify right)
-		)
-	)
-	(hierarchical_label "X_OUT"
-		(shape input)
-		(at 45.72 31.75 90)
-		(effects
-			(font
-				(size 1.27 1.27)
-			)
-			(justify left)
-		)
-	)
-	(hierarchical_label "SAO"
-		(shape input)
-		(at 59.69 162.56 270)
-		(effects
-			(font
-				(size 1.27 1.27)
-			)
-			(justify right)
-		)
-	)

Commit message: Actualizacion PCB Principal
Parts:
- removed C4, C5: C, symbol Device:C
- removed R1: R, symbol Device:R
- added C4, C5: 22p, symbol Device:C_Polarized_Small_US
- C1, C2: value C -> 0.1u
- C3: value C -> 100n
- R1: renamed from R2; value R -> 10k
- R5: value R -> 10k
- Y1: value Crystal -> 32.768kHz
Connections:
- net SA0 is gone; now on net GND: IC3.17 (SA0/H_MOSI_), R1.2
- net GND: now also C4.2, C5.2
- net IMU_BOOTN: now also R5.2
- net IMU_INT: no longer R5.2
- net X_IN: now also C5.1
- net X_OUT: now also C4.1
Other:
- moved on the sheet: C1, C2, R1, R3, R4, R5

Commit message: Actualizacion PCB Principal
Parts:
- removed C3: 100n, symbol Device:C
- added C3: 100n, symbol Device:C_Polarized_Small_US
- C4, C5: value 22p -> C
Connections:
- net CAP: now also C3.1
- net GND: now also C3.2
Other:
- moved on the sheet: C4, C5, R3, R4, R5, Y1

Commit message: actualizacion de pcb
Other:
- note added: "SA0"

Commit message: actualizacion pcb principal
Parts:
- C4, C5: value C -> 22p
- R3, R4: value R -> 4k
Other:
- moved on the sheet: C3, Y1
Changed lines of the file:
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@@
 		)
 	)
-	(text_box "Using a crystal with tolerance 50ppm with 12.5pF (CL) capacitor loading.\nPage 10\n\nCL = (C1.C2)/(C1+C2) + Cpcb"
+	(text_box "Using a crystal with tolerance 50ppm with 12.5pF (CL) capacitor loading.\nPage 10\n"
 		(exclude_from_sim no)
 		(at 12.6999 52.0699 0)
@@
 	(wire
 		(pts
-			(xy 157.48 41.91) (xy 157.48 44.45)
+			(xy 156.21 33.02) (xy 156.21 35.56)
 		)
 		(stroke
@@
 	(wire
 		(pts
-			(xy 39.37 26.67) (xy 45.72 26.67)
+			(xy 38.1 26.67) (xy 45.72 26.67)
 		)
 		(stroke
@@
 	(wire
 		(pts
-			(xy 31.75 26.67) (xy 24.13 26.67)
+			(xy 30.48 26.67) (xy 24.13 26.67)
 		)
 		(stroke
@@
 	(wire
 		(pts
-			(xy 157.48 33.02) (xy 157.48 36.83)
+			(xy 156.21 24.13) (xy 156.21 27.94)
 		)
 		(stroke
@@
 	)
 	(label "CAP"
-		(at 157.48 33.02 0)
+		(at 156.21 24.13 0)
 		(effects
 			(font
@@
 			)
 		)
-		(property "Value" "R"
+		(property "Value" "4k"
 			(at 96.52 35.5599 0)
 			(effects
@@
 	(symbol
 		(lib_id "Device:C_Polarized_Small_US")
-		(at 157.48 39.37 0)
+		(at 156.21 30.48 0)
 		(unit 1)
 		(exclude_from_sim no)
@@
 		(fields_autoplaced yes)
 		(property "Reference" "C3"
-			(at 160.02 37.6681 0)
+			(at 158.75 28.7781 0)
 			(effects
 				(font
@@
 		)
 		(property "Value" "100n"
-			(at 160.02 40.2081 0)
+			(at 158.75 31.3181 0)
 			(effects
 				(font
@@
 		)
 		(property "Footprint" ""
-			(at 157.48 39.37 0)
+			(at 156.21 30.48 0)
 			(effects
 				(font
@@
 		)
 		(property "Datasheet" "~"
-			(at 157.48 39.37 0)
+			(at 156.21 30.48 0)
 			(effects
 				(font
@@
 		)
 		(property "Description" "Polarized capacitor, small US symbol"
-			(at 157.48 39.37 0)
+			(at 156.21 30.48 0)
 			(effects
 				(font
@@
 			)
 		)
-		(property "Value" "C"
+		(property "Value" "22p"
 			(at 26.67 33.8581 0)
 			(effects
@@
 			)
 		)
-		(property "Value" "R"
+		(property "Value" "4k"
 			(at 87.63 35.5599 0)
 			(effects
@@
 			)
 		)
-		(property "Value" "C"
+		(property "Value" "22p"
 			(at 48.26 33.8581 0)
 			(effects
@@
 	(symbol
 		(lib_id "power:GND")
-		(at 157.48 44.45 0)
+		(at 156.21 35.56 0)
 		(unit 1)
 		(exclude_from_sim no)
@@
 		(fields_autoplaced yes)
 		(property "Reference" "#PWR04"
-			(at 157.48 50.8 0)
+			(at 156.21 41.91 0)
 			(effects
 				(font
@@
 		)
 		(property "Value" "GND"
-			(at 157.48 49.53 0)
+			(at 156.21 40.64 0)
 			(effects
 				(font
@@
 		)
 		(property "Footprint" ""
-			(at 157.48 44.45 0)
+			(at 156.21 35.56 0)
 			(effects
 				(font
@@
 		)
 		(property "Datasheet" ""
-			(at 157.48 44.45 0)
+			(at 156.21 35.56 0)
 			(effects
 				(font
@@
 		)
 		(property "Description" "Power symbol creates a global label with name \"GND\" , ground"
-			(at 157.48 44.45 0)
+			(at 156.21 35.56 0)
 			(effects
 				(font
@@
 	(symbol
 		(lib_id "Device:Crystal")
-		(at 35.56 26.67 0)
+		(at 34.29 26.67 0)
 		(unit 1)
 		(exclude_from_sim no)
@@
 		(fields_autoplaced yes)
 		(property "Reference" "Y1"
-			(at 35.56 19.05 0)
+			(at 34.29 19.05 0)
 			(effects
 				(font
@@
 		)
 		(property "Value" "32.768kHz"
-			(at 35.56 21.59 0)
+			(at 34.29 21.59 0)
 			(effects
 				(font
@@
 		)
 		(property "Footprint" ""
-			(at 35.56 26.67 0)
+			(at 34.29 26.67 0)
 			(effects
 				(font
@@
 		)
 		(property "Datasheet" "~"
-			(at 35.56 26.67 0)
+			(at 34.29 26.67 0)
 			(effects
 				(font
@@
 		)
 		(property "Description" "Two pin crystal"
-			(at 35.56 26.67 0)
-			(effects
-				(font
+			(at 34.29 26.67 0)
+			(effects
+				(font

Commit message: Actualizacion de Footprints Resistencias y Capacitores Main PCB
Parts:
- C1, C2, C3, C4, C5: footprint (none) -> Capacitor_SMD:C_0805_2012Metric_Pad1.18x1.45mm_HandSolder
- R1, R3, R4, R5: footprint (none) -> Resistor_SMD:R_0805_2012Metric_Pad1.20x1.40mm_HandSolder
- Y1: footprint (none) -> ABS07:ABS07
Changed lines of the file:
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@@
 			)
 		)
-		(property "Footprint" ""
+		(property "Footprint" "Resistor_SMD:R_0805_2012Metric_Pad1.20x1.40mm_HandSolder"
 			(at 184.912 34.29 90)
 			(effects
@@
 			)
 		)
-		(property "Footprint" ""
+		(property "Footprint" "Capacitor_SMD:C_0805_2012Metric_Pad1.18x1.45mm_HandSolder"
 			(at 200.3552 31.75 0)
 			(effects
@@
 			)
 		)
-		(property "Footprint" ""
+		(property "Footprint" "Resistor_SMD:R_0805_2012Metric_Pad1.20x1.40mm_HandSolder"
 			(at 92.202 34.29 90)
 			(effects
@@
 			)
 		)
-		(property "Footprint" ""
+		(property "Footprint" "Capacitor_SMD:C_0805_2012Metric_Pad1.18x1.45mm_HandSolder"
 			(at 156.21 30.48 0)
 			(effects
@@
 			)
 		)
-		(property "Footprint" ""
+		(property "Footprint" "Capacitor_SMD:C_0805_2012Metric_Pad1.18x1.45mm_HandSolder"
 			(at 24.13 33.02 0)
 			(effects
@@
 			)
 		)
-		(property "Footprint" ""
+		(property "Footprint" "Resistor_SMD:R_0805_2012Metric_Pad1.20x1.40mm_HandSolder"
 			(at 101.092 34.29 90)
 			(effects
@@
 			)
 		)
-		(property "Footprint" ""
+		(property "Footprint" "Resistor_SMD:R_0805_2012Metric_Pad1.20x1.40mm_HandSolder"
 			(at 83.312 34.29 90)
 			(effects
@@
 			)
 		)
-		(property "Footprint" ""
+		(property "Footprint" "Capacitor_SMD:C_0805_2012Metric_Pad1.18x1.45mm_HandSolder"
 			(at 210.5152 31.75 0)
 			(effects
@@
 			)
 		)
-		(property "Footprint" ""
+		(property "Footprint" "Capacitor_SMD:C_0805_2012Metric_Pad1.18x1.45mm_HandSolder"
 			(at 45.72 33.02 0)
 			(effects
@@
 			)
 		)
-		(property "Footprint" ""
+		(property "Footprint" "ABS07:ABS07"
 			(at 34.29 26.67 0)
 			(effects
