File: Hardware/PCB/PCB/Solar_Tracker_PCB_Main/Solar_Tracker_PCB_Main.kicad_pcb (KiCad board)
At the start: 4 copper layers, 94 x 96.5 mm, 67 parts, among them IC1 ESP32-S3-WROOM-1-N4R8, IC2 TPS54302DDCT, IC3 BNO085, IC4 PCF2131TFY, IC6 TLV76133DCYR, J1 SM08B-SRSS-TB_LF__SN_, J2 USB4940-00-A, J3 Conn_01x06_Pin, J4 1977223-1, J5 1977223-1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

Commit message: actualizacion pcb main
Routing:
- net VDD: track 50.0 -> 53.5 mm, vias 22 -> 21
- net J6_6: track 76.9 -> 73.6 mm
- net J6_5: track 78.2 -> 75.4 mm
- net J1_2: track 71.9 -> 74.6 mm
- net J1_3: track 74.4 -> 76.9 mm
- net J6_4: track 79.3 -> 77.3 mm
- net J1_4: track 76.8 -> 78.9 mm
- net GND: track 92.0 -> 94.0 mm, vias 173 -> 208
- net J6_7: track 75.7 -> 74.0 mm
- net J1_5: track 79.2 -> 80.7 mm
- net J1_6: track 81.4 -> 82.7 mm
- net J1_7: track 83.4 -> 84.4 mm
- net J6_3: track 57.5 -> 58.1 mm

Commit message: cambios menores
Routing:
- net GND: track 94.0 -> 98.6 mm, vias 208 -> 206
Changed lines of the file:
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@@
 		(sheetname "/MCU/")
 		(sheetfile "MCU.kicad_sch")
-		(attr through_hole)
+		(attr smd)
 		(fp_line
 			(start -4.47 3.678)
@@
 	)
 	(segment
+		(start 82.3175 99.46)
+		(end 82.3175 101.49)
+		(width 0.2)
+		(layer "F.Cu")
+		(net 69)
+	)
+	(segment
 		(start 120.35 75.36)
 		(end 120.45 75.46)
@@
 	)
 	(segment
-		(start 83.62 101.51)
-		(end 82.2375 101.51)
-		(width 0.2)
-		(layer "F.Cu")
-		(net 69)
-	)
-	(segment
 		(start 86.6 75.97)
 		(end 87.895 75.97)
@@
 	)
 	(segment
+		(start 77.554 102.516)
+		(end 77.538 102.5)
+		(width 0.2)
+		(layer "F.Cu")
+		(net 69)
+	)
+	(segment
 		(start 129.29 48.41)
 		(end 129.29 49.87625)
@@
 	)
 	(segment
+		(start 81.2915 102.516)
+		(end 77.554 102.516)
+		(width 0.2)
+		(layer "F.Cu")
+		(net 69)
+	)
+	(segment
 		(start 81.19 63.88)
 		(end 81.25 63.94)
@@
 	)
 	(segment
-		(start 83.62 99.47)
-		(end 82.3275 99.47)
-		(width 0.2)
-		(layer "F.Cu")
-		(net 69)
-	)
-	(segment
 		(start 122.8 90.7)
 		(end 122.8 91.9625)
@@
 	)
 	(segment
+		(start 82.3175 101.49)
+		(end 81.2915 102.516)
+		(width 0.2)
+		(layer "F.Cu")
+		(net 69)
+	)
+	(segment
 		(start 149.25 63.81375)
 		(end 149.28 63.78375)
@@
 	)
 	(via
-		(at 83.62 99.47)
-		(size 0.7)
-		(drill 0.3)
-		(layers "F.Cu" "B.Cu")
-		(net 69)
-	)
-	(via
 		(at 117.6 58.38)
 		(size 0.7)
@@
 		(size 0.7)
 		(drill 0.3)
-		(layers "F.Cu" "B.Cu")
-		(net 69)
-	)
-	(via
-		(at 83.62 101.51)
-		(size 0.7)
-		(drill 0.3)
