File: Hardware/PCB/PCB/Solar_Tracker_PCB_Main/buck.kicad_sch (KiCad schematic)
At the start: 20 parts, among them IC2 TPS54302DDCT, J7 TB002-500-02BE, Q1 DMP2045U-7, Q2 DMP2045U-7

Commit message: Correccion del esquematico BUCK
Connections:
- net at C8.2, IC2.6 (BOOT): no longer L3.1
- net at C8.1, IC2.2 (SW): now also L3.1
Changed lines of the file:
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@@
+	)
+	(junction
+		(at 102.87 68.58)
+		(diameter 0)
+		(color 0 0 0 0)
 	)
 	(junction
@@
 	)
 	(junction
-		(at 140.97 68.58)
-		(diameter 0)
-		(color 0 0 0 0)
-	)
-	(junction
 		(at 175.26 88.9)
 		(diameter 0)
@@
 	(wire
 		(pts
+			(xy 140.97 54.61) (xy 102.87 54.61)
+		)
+		(stroke
+			(width 0)
+			(type default)
+		)
+	)
+	(wire
+		(pts
 			(xy 100.33 88.9) (xy 111.76 88.9)
 		)
@@
 	(wire
 		(pts
+			(xy 102.87 54.61) (xy 102.87 68.58)
+		)
+		(stroke
+			(width 0)
+			(type default)
+		)
+	)
+	(wire
+		(pts
 			(xy 175.26 68.58) (xy 189.23 68.58)
 		)
@@
 		)
 		(stroke
-			(width 0)
-			(type default)
-		)
-	)
-	(wire
-		(pts
-			(xy 140.97 54.61) (xy 140.97 68.58)
-		)
-		(stroke
